Commit message: Update mech2bot_description.urdf

File: src/description/mech2bot_description.urdf (robot description, URDF)
Before this commit: robot mech2bot, 2 links, 1 joints
Links:
- added link lidar_link, mass 0.19; collision cylinder length=0.055 radius=0.0508; visual cylinder length=0.055 radius=0.0508
Joints:
- added joint lidar_joint: type fixed, parent base_link, child lidar_link, origin xyz=0 0 0.12 rpy=0 0 0

Commit message: Update mech2bot_description.urdf

File: src/description/mech2bot_description.urdf (robot description, URDF)
Before this commit: robot mech2bot, 3 links, 2 joints
Links:
- link lidar_link: geometry collision cylinder length=0.051 radius=0.0484; visual cylinder length=0.051 radius=0.0484
Joints:
- joint lidar_joint: origin xyz=0 0 0.12 rpy=0 0 0 -> xyz=0 0 0.0572 rpy=0 0 0
